Commit message: adding pen

File: mengine/assets/pen/pen.urdf (robot description, URDF)
Before this commit: robot pen, 1 links, 0 joints
Links:
- removed link base_link
- added link pen_body, mass 0.95; collision box size=0.02 0.02 0.10; visual box size=0.02 0.02 0.10
- added link pen_tip, mass 0.05; collision sphere radius=0.015; visual sphere radius=0.015
Joints:
- added joint pen_joint: type fixed, parent pen_body, child pen_tip, origin xyz=0 0 -0.05 rpy=0 0 0
